Commit message: done

File: body.urdf (robot description, URDF)
Before this commit: robot robot, 3 links, 2 joints
Links:
- added link LeftLeg, mass 1; collision box size=1 0.2 0.2; visual box size=1 0.2 0.2
- added link LowerBackLeg, mass 1; collision box size=0.2 0.2 1; visual box size=0.2 0.2 1
- added link LowerFrontLeg, mass 1; collision box size=0.2 0.2 1; visual box size=0.2 0.2 1
- added link LowerLeftLeg, mass 1; collision box size=0.2 0.2 1; visual box size=0.2 0.2 1
- added link LowerRightLeg, mass 1; collision box size=0.2 0.2 1; visual box size=0.2 0.2 1
- added link RightLeg, mass 1; collision box size=1 0.2 0.2; visual box size=1 0.2 0.2
- link BackLeg: geometry collision box size=0.2 1 0.2; visual box size=0.2 1 0.2
- link FrontLeg: geometry collision box size=0.2 1 0.2; visual box size=0.2 1 0.2
Joints:
- added joint BackLeg_LowerBackLeg: type revolute, parent BackLeg, child LowerBackLeg, origin xyz=0 -1 0 rpy=0 0 0, axis 1 0 0, limit lower=-3.14159 upper=3.14159 effort=0.0 velocity=0.0
- added joint FrontLeg_LowerFrontLeg: type revolute, parent FrontLeg, child LowerFrontLeg, origin xyz=0 1 0 rpy=0 0 0, axis 1 0 0, limit lower=-3.14159 upper=3.14159 effort=0.0 velocity=0.0
- added joint LeftLeg_LowerLeftLeg: type revolute, parent LeftLeg, child LowerLeftLeg, origin xyz=1 0 0 rpy=0 0 0, axis 0 1 0, limit lower=-3.14159 upper=3.14159 effort=0.0 velocity=0.0
- added joint RightLeg_LowerRightLeg: type revolute, parent RightLeg, child LowerRightLeg, origin xyz=-1 0 0 rpy=0 0 0, axis 0 1 0, limit lower=-3.14159 upper=3.14159 effort=0.0 velocity=0.0
- added joint Torso_LeftLeg: type revolute, parent Torso, child LeftLeg, origin xyz=0.5 0 1 rpy=0 0 0, axis 0 1 0, limit lower=-3.14159 upper=3.14159 effort=0.0 velocity=0.0
- added joint Torso_RightLeg: type revolute, parent Torso, child RightLeg, origin xyz=-0.5 0 1 rpy=0 0 0, axis 0 1 0, limit lower=-3.14159 upper=3.14159 effort=0.0 velocity=0.0
- joint Torso_BackLeg: axis 0 1 0 -> 1 0 0; origin xyz=0.5 0 1 rpy=0 0 0 -> xyz=0 -0.5 1 rpy=0 0 0
- joint Torso_FrontLeg: axis 0 1 0 -> 1 0 0; origin xyz=-0.5 0 1 rpy=0 0 0 -> xyz=0 0.5 1 rpy=0 0 0

Commit message: asd

File: body.urdf (robot description, URDF)
Before this commit: robot robot, 9 links, 8 joints
Links:
- removed link BackLeg
- removed link FrontLeg
- removed link LeftLeg
- removed link LowerBackLeg
- removed link LowerFrontLeg
- removed link LowerLeftLeg
- removed link LowerRightLeg
- removed link RightLeg
- added link FrontLeftLeg, mass 1; collision box size=0.2 0.2 0.7; visual box size=0.2 0.2 0.7
- link Torso: geometry collision box size=3 1.5 0.6; visual box size=3 1.5 0.6
Joints:
- removed joint BackLeg_LowerBackLeg
- removed joint FrontLeg_LowerFrontLeg
- removed joint LeftLeg_LowerLeftLeg
- removed joint RightLeg_LowerRightLeg
- removed joint Torso_BackLeg
- removed joint Torso_FrontLeg
- removed joint Torso_LeftLeg
- removed joint Torso_RightLeg
- added joint Torso_FrontLeftLeg: type revolute, parent Torso, child FrontLeftLeg, origin xyz=-1 -1 0.7 rpy=0 0 0, axis 0 1 0, limit lower=-3.14159 upper=3.14159 effort=0.0 velocity=0.0

Commit message: Deliberable 01

File: body.urdf (robot description, URDF)
Before this commit: robot robot, 2 links, 1 joints
Links:
- removed link FrontLeftLeg
- added link BackLeftDownLeg, mass 1; collision box size=0.2 0.2 0.6; visual box size=0.2 0.2 0.6
- added link BackLeftFoot, mass 1; collision box size=0.4 0.2 0.1; visual box size=0.4 0.2 0.1
- added link BackLeftSide, mass 1; collision box size=0.3 0.3 0.3; visual box size=0.3 0.3 0.3
- added link BackLeftUpLeg, mass 1; collision box size=0.3 0.3 0.5; visual box size=0.3 0.3 0.5
- added link BackRightDownLeg, mass 1; collision box size=0.2 0.2 0.6; visual box size=0.2 0.2 0.6
- added link BackRightFoot, mass 1; collision box size=0.4 0.2 0.1; visual box size=0.4 0.2 0.1
- added link BackRightSide, mass 1; collision box size=0.3 0.3 0.3; visual box size=0.3 0.3 0.3
- added link BackRightUpLeg, mass 1; collision box size=0.3 0.3 0.5; visual box size=0.3 0.3 0.5
- added link FrontLeftDownLeg, mass 1; collision box size=0.2 0.2 0.6; visual box size=0.2 0.2 0.6
- added link FrontLeftFoot, mass 1; collision box size=0.4 0.2 0.1; visual box size=0.4 0.2 0.1
- added link FrontLeftSide, mass 1; collision box size=0.3 0.3 0.3; visual box size=0.3 0.3 0.3
- added link FrontLeftUpLeg, mass 1; collision box size=0.3 0.3 0.5; visual box size=0.3 0.3 0.5
- added link FrontRightDownLeg, mass 1; collision box size=0.2 0.2 0.6; visual box size=0.2 0.2 0.6
- added link FrontRightFoot, mass 1; collision box size=0.4 0.2 0.1; visual box size=0.4 0.2 0.1
- added link FrontRightSide, mass 1; collision box size=0.3 0.3 0.3; visual box size=0.3 0.3 0.3
- added link FrontRightUpLeg, mass 1; collision box size=0.3 0.3 0.5; visual box size=0.3 0.3 0.5
Joints:
- removed joint Torso_FrontLeftLeg
- added joint BackLeftDownLeg_BackLeftFoot: type revolute, parent BackLeftDownLeg, child BackLeftFoot, origin xyz=0.1 0 -0.6 rpy=0 0 0, axis 1 0 0, limit lower=-3.14159 upper=3.14159 effort=0.0 velocity=0.0
- added joint BackLeftSide_BackLeftUpLeg: type revolute, parent BackLeftSide, child BackLeftUpLeg, origin xyz=0.15 -0.15 -0.15 rpy=0 0 0, axis 0 1 0, limit lower=-3.14159 upper=3.14159 effort=0.0 velocity=0.0
- added joint BackLeftUpLeg_BackLeftDownLeg: type revolute, parent BackLeftUpLeg, child BackLeftDownLeg, origin xyz=0.3 0 -0.5 rpy=0 0 0, axis 0 1 0, limit lower=-3.14159 upper=3.14159 effort=0.0 velocity=0.0
- added joint BackRightDownLeg_BackRightFoot: type revolute, parent BackRightDownLeg, child BackRightFoot, origin xyz=0.1 0 -0.6 rpy=0 0 0, axis 1 0 0, limit lower=-3.14159 upper=3.14159 effort=0.0 velocity=0.0
- added joint BackRightSide_BackRightUpLeg: type revolute, parent BackRightSide, child BackRightUpLeg, origin xyz=0.15 0.15 -0.15 rpy=0 0 0, axis 0 1 0, limit lower=-3.14159 upper=3.14159 effort=0.0 velocity=0.0
- added joint BackRightUpLeg_BackRightDownLeg: type revolute, parent BackRightUpLeg, child BackRightDownLeg, origin xyz=0.3 0 -0.5 rpy=0 0 0, axis 0 1 0, limit lower=-3.14159 upper=3.14159 effort=0.0 velocity=0.0
- added joint FrontLeftDownLeg_FrontLeftFoot: type revolute, parent FrontLeftDownLeg, child FrontLeftFoot, origin xyz=0.1 0 -0.6 rpy=0 0 0, axis 1 0 0, limit lower=-3.14159 upper=3.14159 effort=0.0 velocity=0.0
- added joint FrontLeftSide_FrontLeftUpLeg: type revolute, parent FrontLeftSide, child FrontLeftUpLeg, origin xyz=0.15 -0.15 -0.15 rpy=0 0 0, axis 0 1 0, limit lower=-3.14159 upper=3.14159 effort=0.0 velocity=0.0
- added joint FrontLeftUpLeg_FrontLeftDownLeg: type revolute, parent FrontLeftUpLeg, child FrontLeftDownLeg, origin xyz=0.3 0 -0.5 rpy=0 0 0, axis 0 1 0, limit lower=-3.14159 upper=3.14159 effort=0.0 velocity=0.0
- added joint FrontRightDownLeg_FrontRightFoot: type revolute, parent FrontRightDownLeg, child FrontRightFoot, origin xyz=0.1 0 -0.6 rpy=0 0 0, axis 1 0 0, limit lower=-3.14159 upper=3.14159 effort=0.0 velocity=0.0
- added joint FrontRightSide_FrontRightUpLeg: type revolute, parent FrontRightSide, child FrontRightUpLeg, origin xyz=0.15 0.15 -0.15 rpy=0 0 0, axis 0 1 0, limit lower=-3.14159 upper=3.14159 effort=0.0 velocity=0.0
- added joint FrontRightUpLeg_FrontRightDownLeg: type revolute, parent FrontRightUpLeg, child FrontRightDownLeg, origin xyz=0.3 0 -0.5 rpy=0 0 0, axis 0 1 0, limit lower=-3.14159 upper=3.14159 effort=0.0 velocity=0.0
- added joint Torso_BackLeftSide: type revolute, parent Torso, child BackLeftSide, origin xyz=1.3 -0.75 1.3 rpy=0 0 0, axis 0 1 0, limit lower=-3.14159 upper=3.14159 effort=0.0 velocity=0.0
- added joint Torso_BackRightSide: type revolute, parent Torso, child BackRightSide, origin xyz=1.3 0.75 1.3 rpy=0 0 0, axis 0 1 0, limit lower=-3.14159 upper=3.14159 effort=0.0 velocity=0.0
- added joint Torso_FrontLeftSide: type revolute, parent Torso, child FrontLeftSide, origin xyz=-1.3 -0.75 1.3 rpy=0 0 0, axis 0 1 0, limit lower=-3.14159 upper=3.14159 effort=0.0 velocity=0.0
- added joint Torso_FrontRightSide: type revolute, parent Torso, child FrontRightSide, origin xyz=-1.3 0.75 1.3 rpy=0 0 0, axis 0 1 0, limit lower=-3.14159 upper=3.14159 effort=0.0 velocity=0.0
